Commit message: fix orientation of LIDAR

File: linorobot2_description/urdf/4wd_properties.urdf.xacro (robot description, xacro)
@@ -13,5 +13,5 @@
   <xacro:property name="wheel_torque" value="20" />
   <xacro:property name="laser_pose">
-    <origin xyz="0.08 0 0.122" rpy="0 0 0"/>
+    <origin xyz="0.08 0 0.122" rpy="0 0 3.14"/>
   </xacro:property>
   <!-- <xacro:property name="depth_sensor_pose">

Commit message: Add camera (#1)
* make laser rays show up in gazebo

* removed depth camera and added urdf position of webcam

* simulate camera in gazebo

* added camera bringup

* fixed orientation of LIDAR

File: linorobot2_description/urdf/4wd_properties.urdf.xacro (robot description, xacro)
@@ -13,8 +13,11 @@
   <xacro:property name="wheel_torque" value="20" />
   <xacro:property name="laser_pose">
-    <origin xyz="0.08 0 0.122" rpy="0 0 0"/>
+    <origin xyz="0.08 0 0.122" rpy="0 0 3.14"/>
   </xacro:property>
-  <xacro:property name="depth_sensor_pose">
+  <!-- <xacro:property name="depth_sensor_pose">
     <origin xyz="-0.065 0 0.255" rpy="0 0 0"/>
+  </xacro:property> -->
+  <xacro:property name="camera_pose">
+    <origin xyz="0.134 0 0.02" rpy="0 0 0"/>
   </xacro:property>
 </robot>

File: linorobot2_description/urdf/robots/4wd.urdf.xacro (robot description, xacro)
@@ -7,4 +7,5 @@
   <xacro:include filename="$(find linorobot2_description)/urdf/sensors/generic_laser.urdf.xacro" />
   <xacro:include filename="$(find linorobot2_description)/urdf/sensors/depth_sensor.urdf.xacro" />
+  <xacro:include filename="$(find linorobot2_description)/urdf/sensors/camera.urdf.xacro" />
   <xacro:include filename="$(find linorobot2_description)/urdf/controllers/skid_steer.urdf.xacro" />
   <xacro:base
@@ -56,7 +57,10 @@
     <xacro:insert_block name="laser_pose" />
   </xacro:generic_laser>
-  <xacro:depth_sensor>
+  <!-- <xacro:depth_sensor>
     <xacro:insert_block name="depth_sensor_pose" />
-  </xacro:depth_sensor>
+  </xacro:depth_sensor> -->
+  <xacro:camera>
+    <xacro:insert_block name="camera_pose" />
+  </xacro:camera>
   <xacro:diff_drive_controller
     wheel_separation="${wheel_pos_y * 2}"

File: linorobot2_description/urdf/sensors/laser.urdf.xacro (robot description, xacro)
@@ -46,5 +46,5 @@
         <update_rate>${update_rate}</update_rate>
         <pose>0 0 0 0 0 0</pose>
-        <visualize>false</visualize>
+        <visualize>true</visualize>
         <ray>
           <scan>
